File: ergogen/output/pcbs/mulloy42_left.kicad_pcb (KiCad board)
At the start: 2 copper layers, 146.1 x 95.8 mm, 97 parts

Commit message: updated left/right pcb
Parts:
- removed D22, D23, D24, D25, D26, D27, D28, D29, D30, D31, D32, D33, D34, D35, D36, D37, D38, D39, D40, D41, D42: , ComboDiode
- removed MH5, MH6, MH7, MH8: , ceoloide:mounting_hole_npth
- removed S22, S23, S24, S25, S26, S27, S28, S29, S30, S31, S32, S33, S34, S35, S36, S37, S38, S39, S40, S41, S42: , PG1350

Commit message: new config file for mulloy42
Routing:
- net P18: track 0.00 -> 206.5 mm
- net P9: track 0.00 -> 192.7 mm, vias 0 -> 1
- net P5: track 0.00 -> 191.6 mm
- net P4: track 0.00 -> 162.3 mm
- net P8: track 0.00 -> 156.7 mm, vias 0 -> 1
- net P3: track 0.00 -> 155.7 mm
- net P16: track 0.00 -> 147.1 mm, vias 0 -> 5
- net P15: track 0.00 -> 138.0 mm, vias 0 -> 1
- net P2: track 0.00 -> 117.6 mm
- net P10: track 0.00 -> 110.9 mm
- net GND: track 0.00 -> 78.5 mm, vias 0 -> 1
- net RST: track 0.00 -> 59.4 mm
- net RAW: track 0.00 -> 45.5 mm, vias 0 -> 1
- net VCC: track 0.00 -> 28.4 mm
- net inner_thumb: track 0.00 -> 15.4 mm
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
Commit message: final pcb designs and gerber files
Routing:
- net GND: track 78.5 -> 104.8 mm, vias 1 -> 4
- net P10: track 110.9 -> 112.2 mm
- added copper zone on B.Cu, net GND
- added copper zone on F.Cu, net GND

Commit message: updating dxf to make modeling case easier
Parts:
- added D22: , ComboDiode, F.Cu at (393.0, 105.0)
- added D23: , ComboDiode, F.Cu at (393.0, 86.0)
- added D24: , ComboDiode, F.Cu at (393.0, 67.0)
- added D25: , ComboDiode, F.Cu at (373.0, 105.0)
- added D26: , ComboDiode, F.Cu at (373.0, 86.0)
- added D27: , ComboDiode, F.Cu at (373.0, 67.0)
- added D28: , ComboDiode, F.Cu at (353.0, 95.0)
- added D29: , ComboDiode, F.Cu at (353.0, 76.0)
- added D30: , ComboDiode, F.Cu at (353.0, 57.0)
- added D31: , ComboDiode, F.Cu at (333.0, 90.0)
- added D32: , ComboDiode, F.Cu at (333.0, 71.0)
- added D33: , ComboDiode, F.Cu at (333.0, 52.0)
- added D34: , ComboDiode, F.Cu at (313.0, 96.0)
- added D35: , ComboDiode, F.Cu at (313.0, 77.0)
- added D36: , ComboDiode, F.Cu at (313.0, 58.0)
- added D37: , ComboDiode, F.Cu at (293.0, 98.0)
- added D38: , ComboDiode, F.Cu at (293.0, 79.0)
- added D39: , ComboDiode, F.Cu at (293.0, 60.0)
- added D40: , ComboDiode, F.Cu at (313.0, 117.0)
- added D41: , ComboDiode, F.Cu at (293.9, 119.6)
- added D42: , ComboDiode, F.Cu at (266.8, 118.2)
- added MH5: , ceoloide:mounting_hole_npth, F.Cu at (383.0, 71.5)
- added MH6: , ceoloide:mounting_hole_npth, F.Cu at (383.0, 90.5)
- added MH7: , ceoloide:mounting_hole_npth, F.Cu at (303.0, 63.5)
- added MH8: , ceoloide:mounting_hole_npth, F.Cu at (282.3, 104.7)
- added S22: , PG1350, F.Cu at (393.0, 100.0)
- added S23: , PG1350, F.Cu at (393.0, 81.0)
- added S24: , PG1350, F.Cu at (393.0, 62.0)
- added S25: , PG1350, F.Cu at (373.0, 100.0)
- added S26: , PG1350, F.Cu at (373.0, 81.0)
- added S27: , PG1350, F.Cu at (373.0, 62.0)
- added S28: , PG1350, F.Cu at (353.0, 90.0)
- added S29: , PG1350, F.Cu at (353.0, 71.0)
- added S30: , PG1350, F.Cu at (353.0, 52.0)
- added S31: , PG1350, F.Cu at (333.0, 85.0)
- added S32: , PG1350, F.Cu at (333.0, 66.0)
- added S33: , PG1350, F.Cu at (333.0, 47.0)
- added S34: , PG1350, F.Cu at (313.0, 91.0)
- added S35: , PG1350, F.Cu at (313.0, 72.0)
- added S36: , PG1350, F.Cu at (313.0, 53.0)
- added S37: , PG1350, F.Cu at (293.0, 93.0)
- added S38: , PG1350, F.Cu at (293.0, 74.0)
- added S39: , PG1350, F.Cu at (293.0, 55.0)
- added S40: , PG1350, F.Cu at (313.0, 112.0)
- added S41: , PG1350, F.Cu at (293.0, 114.7)
- added S42: , PG1350, F.Cu at (271.5, 116.5)
Routing:
- net P18: track 206.5 -> 0.00 mm
- net P9: track 192.7 -> 0.00 mm, vias 1 -> 0
- net P5: track 191.6 -> 0.00 mm
- net P4: track 162.3 -> 0.00 mm
- net P8: track 156.7 -> 0.00 mm, vias 1 -> 0
- net P3: track 155.7 -> 0.00 mm
- net P16: track 147.1 -> 0.00 mm, vias 5 -> 0
- net P15: track 138.0 -> 0.00 mm, vias 1 -> 0
- net P2: track 117.6 -> 0.00 mm
- net P10: track 112.2 -> 0.00 mm
- net GND: track 104.8 -> 0.00 mm, vias 4 -> 0
- net RST: track 59.4 -> 0.00 mm
- net RAW: track 45.5 -> 0.00 mm, vias 1 -> 0
- net VCC: track 28.4 -> 0.00 mm
- net inner_thumb: track 15.4 -> 0.00 mm
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- removed copper zone on B.Cu, net GND
- removed copper zone on F.Cu, net GND
