File: ergogen/output/pcbs/mulloy42_right.kicad_pcb (KiCad board)
At the start: 2 copper layers, 146.1 x 95.8 mm, 97 parts

Commit message: new config file for mulloy42
Parts:
- removed D1, D10, D11, D12, D13, D14, D15, D16, D17, D18, D19, D2, D20, D21, D3, D4, D5, D6, D7, D8, D9: , ComboDiode
- removed MH1, MH2, MH3, MH4: , ceoloide:mounting_hole_npth
- removed S1, S10, S11, S12, S13, S14, S15, S16, S17, S18, S19, S2, S20, S21, S3, S4, S5, S6, S7, S8, S9: , PG1350
- moved D22 126.3 mm to (269.2, 130.3)
- moved D23 126.3 mm to (269.2, 111.3)
- moved D24 126.3 mm to (269.2, 92.3)
- moved D25 126.3 mm to (249.2, 130.3)
- moved D26 126.3 mm to (249.2, 111.3)
- moved D27 126.3 mm to (249.2, 92.3)
- moved D28 126.3 mm to (229.2, 120.3)
- moved D29 126.3 mm to (229.2, 101.3)
- moved D30 126.3 mm to (229.2, 82.3)
- moved D31 126.3 mm to (209.2, 115.3)
- moved D32 126.3 mm to (209.2, 96.3)
- moved D33 126.3 mm to (209.2, 77.3)
- moved D34 126.3 mm to (189.2, 121.3)
- moved D35 126.3 mm to (189.2, 102.3)
- moved D36 126.3 mm to (189.2, 83.3)
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Connections:
- DISP1 pad 1: DA -> P7
- DISP1 pad 2: CL -> P6
- DISP1 pad 5: CS -> P14
Routing:
- net P8: track 0.00 -> 204.1 mm
- net P9: track 0.00 -> 181.8 mm, vias 0 -> 5
- net P5: track 0.00 -> 178.8 mm, vias 0 -> 2
- net P3: track 0.00 -> 166.2 mm, vias 0 -> 2
- net P4: track 0.00 -> 165.5 mm, vias 0 -> 2
- net P18: track 0.00 -> 134.8 mm, vias 0 -> 1
- net P16: track 0.00 -> 120.1 mm, vias 0 -> 1
- net P15: track 0.00 -> 114.3 mm, vias 0 -> 1
- net P2: track 0.00 -> 105.6 mm, vias 0 -> 2
- net P10: track 0.00 -> 104.9 mm
- net GND: track 0.00 -> 87.9 mm
- net RST: track 0.00 -> 69.2 mm, vias 0 -> 1
- net RAW: track 0.00 -> 63.0 mm, vias 0 -> 1
- net VCC: track 0.00 -> 30.8 mm
- net mirror_index_thumb: track 0.00 -> 15.1 mm
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
Commit message: final pcb designs and gerber files
Parts:
- moved D41 16.6 mm to (183.1, 155.2)
- moved S41 16.6 mm to (182.2, 150.3)
- moved D22 16.6 mm to (282.2, 140.6)
- moved D23 16.6 mm to (282.2, 121.6)
- moved D24 16.6 mm to (282.2, 102.6)
- moved D25 16.6 mm to (262.2, 140.6)
- moved D26 16.6 mm to (262.2, 121.6)
- moved D27 16.6 mm to (262.2, 102.6)
- moved D28 16.6 mm to (242.2, 130.6)
- moved D29 16.6 mm to (242.2, 111.6)
- moved D30 16.6 mm to (242.2, 92.6)
- moved D31 16.6 mm to (222.2, 125.6)
- moved D32 16.6 mm to (222.2, 106.6)
- moved D33 16.6 mm to (222.2, 87.6)
- moved D34 16.6 mm to (202.2, 131.6)
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Routing:
- net P8: track 204.1 -> 154.3 mm, vias 0 -> 1
- net RST: track 69.2 -> 85.4 mm, vias 1 -> 0
- net GND: track 87.9 -> 77.7 mm
- net P9: track 181.8 -> 176.0 mm, vias 5 -> 1
- net P3: track 166.2 -> 161.1 mm
- net P15: track 114.3 -> 109.6 mm
- net RAW: track 63.0 -> 59.6 mm, vias 1 -> 0
- net P10: track 104.9 -> 108.3 mm
- net P2: track 105.6 -> 102.4 mm, vias 2 -> 0
- net P18: track 134.8 -> 132.3 mm
- net P16: track 120.1 -> 118.5 mm
- net P5: track 178.8 -> 180.0 mm
- net VCC: track 30.8 -> 31.8 mm, vias 0 -> 1
- net P4: track 165.5 -> 166.3 mm
- net P14: vias 0 -> 1
- added copper zone on B.Cu, net GND
- added copper zone on F.Cu, net GND

Commit message: updating dxf to make modeling case easier
Parts:
- added D1: , ComboDiode, F.Cu at (100.0, 105.0)
- added D10: , ComboDiode, F.Cu at (160.0, 90.0)
- added D11: , ComboDiode, F.Cu at (160.0, 71.0)
- added D12: , ComboDiode, F.Cu at (160.0, 52.0)
- added D13: , ComboDiode, F.Cu at (180.0, 96.0)
- added D14: , ComboDiode, F.Cu at (180.0, 77.0)
- added D15: , ComboDiode, F.Cu at (180.0, 58.0)
- added D16: , ComboDiode, F.Cu at (200.0, 98.0)
- added D17: , ComboDiode, F.Cu at (200.0, 79.0)
- added D18: , ComboDiode, F.Cu at (200.0, 60.0)
- added D19: , ComboDiode, F.Cu at (180.0, 117.0)
- added D2: , ComboDiode, F.Cu at (100.0, 86.0)
- added D20: , ComboDiode, F.Cu at (199.1, 119.6)
- added D21: , ComboDiode, F.Cu at (226.2, 118.2)
- added D3: , ComboDiode, F.Cu at (100.0, 67.0)
- added D4: , ComboDiode, F.Cu at (120.0, 105.0)
- added D5: , ComboDiode, F.Cu at (120.0, 86.0)
- added D6: , ComboDiode, F.Cu at (120.0, 67.0)
- added D7: , ComboDiode, F.Cu at (140.0, 95.0)
- added D8: , ComboDiode, F.Cu at (140.0, 76.0)
- added D9: , ComboDiode, F.Cu at (140.0, 57.0)
- added MH1: , ceoloide:mounting_hole_npth, F.Cu at (110.0, 71.5)
- added MH2: , ceoloide:mounting_hole_npth, F.Cu at (110.0, 90.5)
- added MH3: , ceoloide:mounting_hole_npth, F.Cu at (190.0, 63.5)
- added MH4: , ceoloide:mounting_hole_npth, F.Cu at (210.8, 104.7)
- added S1: , PG1350, F.Cu at (100.0, 100.0)
- added S10: , PG1350, F.Cu at (160.0, 85.0)
- added S11: , PG1350, F.Cu at (160.0, 66.0)
- added S12: , PG1350, F.Cu at (160.0, 47.0)
- added S13: , PG1350, F.Cu at (180.0, 91.0)
- added S14: , PG1350, F.Cu at (180.0, 72.0)
- added S15: , PG1350, F.Cu at (180.0, 53.0)
- added S16: , PG1350, F.Cu at (200.0, 93.0)
- added S17: , PG1350, F.Cu at (200.0, 74.0)
- added S18: , PG1350, F.Cu at (200.0, 55.0)
- added S19: , PG1350, F.Cu at (180.0, 112.0)
- added S2: , PG1350, F.Cu at (100.0, 81.0)
- added S20: , PG1350, F.Cu at (200.0, 114.7)
- added S21: , PG1350, F.Cu at (221.5, 116.5)
- added S3: , PG1350, F.Cu at (100.0, 62.0)
- added S4: , PG1350, F.Cu at (120.0, 100.0)
- added S5: , PG1350, F.Cu at (120.0, 81.0)
- added S6: , PG1350, F.Cu at (120.0, 62.0)
- added S7: , PG1350, F.Cu at (140.0, 90.0)
- added S8: , PG1350, F.Cu at (140.0, 71.0)
- added S9: , PG1350, F.Cu at (140.0, 52.0)
- moved D22 116.4 mm to (393.0, 105.0)
- moved D23 116.4 mm to (393.0, 86.0)
- moved D24 116.4 mm to (393.0, 67.0)
- moved D25 116.4 mm to (373.0, 105.0)
- moved D26 116.4 mm to (373.0, 86.0)
- moved D27 116.4 mm to (373.0, 67.0)
- moved D28 116.4 mm to (353.0, 95.0)
- moved D29 116.4 mm to (353.0, 76.0)
- moved D30 116.4 mm to (353.0, 57.0)
- moved D31 116.4 mm to (333.0, 90.0)
- moved D32 116.4 mm to (333.0, 71.0)
- moved D33 116.4 mm to (333.0, 52.0)
- moved D34 116.4 mm to (313.0, 96.0)
- moved D35 116.4 mm to (313.0, 77.0)
- moved D36 116.4 mm to (313.0, 58.0)
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Routing:
- net P5: track 180.0 -> 0.00 mm, vias 2 -> 0
- net P9: track 176.0 -> 0.00 mm, vias 1 -> 0
- net P4: track 166.3 -> 0.00 mm, vias 2 -> 0
- net P3: track 161.1 -> 0.00 mm, vias 2 -> 0
- net P8: track 154.3 -> 0.00 mm, vias 1 -> 0
- net P18: track 132.3 -> 0.00 mm, vias 1 -> 0
- net P16: track 118.5 -> 0.00 mm, vias 1 -> 0
- net P15: track 109.6 -> 0.00 mm, vias 1 -> 0
- net P10: track 108.3 -> 0.00 mm
- net P2: track 102.4 -> 0.00 mm
- net RST: track 85.4 -> 0.00 mm
- net GND: track 77.7 -> 0.00 mm
- net RAW: track 59.6 -> 0.00 mm
- net VCC: track 31.8 -> 0.00 mm, vias 1 -> 0
- net mirror_index_thumb: track 15.1 -> 0.00 mm
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- removed copper zone on B.Cu, net GND
- removed copper zone on F.Cu, net GND
